Commit message: feat(miniarm): enable gazebo

File: src/miniarm/config/miniarm.ros2_control.xacro (robot description, xacro)
@@ -1,10 +1,14 @@
 <?xml version="1.0"?>
 <robot xmlns:xacro="http://www.ros.org/wiki/xacro">
-    <xacro:macro name="simple_arm_ros2_control" params="name initial_positions_file">
-        <xacro:property name="initial_positions" value="${load_yaml(initial_positions_file)['initial_positions']}"/>
-        <ros2_control name="${name}" type="system">
+    <xacro:macro name="miniarm_ros2_control" params="name initial_positions_file">
+        <xacro:property name="initial_positions" value="${xacro.load_yaml(initial_positions_file)['initial_positions']}"/>
+        <link name="world"/>
+        <joint name="fixed" type="fixed">
+            <parent link="world"/>
+            <child link="base_link"/>
+        </joint>
+        <ros2_control name="GazeboSystem" type="system">
             <hardware>
-                <!-- By default, set up controllers for simulation. This won't work on real hardware -->
-                <plugin>mock_components/GenericSystem</plugin>
+              <plugin>gazebo_ros2_control/GazeboSystem</plugin>
             </hardware>
             <joint name="yaw_link">
@@ -51,4 +55,11 @@
             </joint>
         </ros2_control>
+        <gazebo>
+          <plugin filename="libgazebo_ros2_control.so" name="gazebo_ros2_control">
+              <parameters>$(find miniarm)/config/ros2_controllers.yaml</parameters>
+              <robot_param>robot_description</robot_param>
+              <robot_param_node>robot_state_publisher</robot_param_node>
+          </plugin>
+        </gazebo>
     </xacro:macro>
 </robot>
