Commit message: feat(simple): [M] update launch

File: src/simple_arm/urdf/simple_arm.urdf (robot description, URDF)
Before this commit: robot simple_arm, 7 links, 6 joints
Links:
- added link world; visual box size=0.001 0.001 0.001
Joints:
- added joint world_joint: type fixed, parent world, child base_link
